File: mic-array.sch (KiCad schematic (older format))
At the start: 14 parts, among them J1 CON40A, K1 74LV244

Commit message: Add new PCB design with improved constraints and routing. Change connector type to 2.54mm one.
Parts:
- J1: footprint Connector_PinSocket_1.27mm:PinSocket_2x20_P1.27mm_Vertical -> Connector_PinSocket_2.54mm:PinSocket_2x20_P2.54mm_Vertical
Changed lines of the file:
@@
 EESchema Schematic File Version 4
-LIBS:mic-array-cache
 EELAYER 26 0
 EELAYER END
@@
 F 0 "J1" H 8550 2967 50  0000 C CNN
 F 1 "CON40A" H 8550 2876 50  0000 C CNN
-F 2 "Connector_PinSocket_1.27mm:PinSocket_2x20_P1.27mm_Vertical" H 8500 1850 50  0001 C CNN
+F 2 "Connector_PinSocket_2.54mm:PinSocket_2x20_P2.54mm_Vertical" H 8500 1850 50  0001 C CNN
 F 3 "~" H 8500 1850 50  0001 C CNN
 	1    8500 1850

Commit message: Add a new buffer to compensate nets impedance.
Parts:
- removed RN1, RN2, RN3, RN4, RN5, RN6, RN7: 0, bridges:bridge_1x4_0.1mm, symbol Device:R_Network04
- added C2: 100n, Capacitor_SMD:C_0603_1608Metric_Pad1.05x0.95mm_HandSolder, symbol Device:C_Small
- added K2: 74LV244, Package_SO:SSOP-20_4.4x6.5mm_P0.65mm, symbol 74xx:74HC244
- added NT1, NT10, NT11, NT12, NT13, NT14, NT2, NT3, NT4, NT5, NT6, NT7, NT8, NT9: Tie, bridges:bridge_1x2_0.12mm, symbol Device:Net-Tie_3_Tee
- renumbered C5 to C1, C1 to C3, C2 to C4, C3 to C5, C4 to C6
Connections:
- net labels added: CLK10, CLK10_0, CLK10_1, CLK11, CLK11_0, CLK11_1, CLK12, CLK12_0, CLK12_1, CLK13, CLK13_0, CLK13_1, CLK7, CLK7_0, CLK7_1, CLK8, CLK8_0, CLK8_1, CLK9, CLK9_0, CLK9_1
- net labels removed: CLK0_2, CLK0_3, CLK1_2, CLK1_3, CLK2_2, CLK2_3, CLK3_2, CLK3_3, CLK4_2, CLK4_3, CLK5_2, CLK5_3, CLK6_2, CLK6_3
- wire segments 34 -> 58
- no-connect marks 23 -> 24
Other:
- moved on the sheet: C3, C4, C5, C6
