File: mic_pair.sch (KiCad schematic (older format))
At the start: 4 parts, among them U1 MIC, U2 MIC

Commit message: Add a new buffer to compensate nets impedance.
Parts:
- renumbered C6 to C7, C7 to C8
